File: electronics/view_base/view_base.kicad_sch (KiCad schematic)
At the start: 108 parts, among them J1 BLDC, J2 USB_C_Receptacle_USB2.0, J3 LCD, J4 A, J5 B, J6 Conn_01x28_Socket, J7 Conn_01x28_Socket, J8 Conn_01x03_Socket, J9 Conn_01x04_Socket, Q1 MMBT4403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

Commit message: sunday work
Parts:
- removed TP15: TX, Modified:TestPoint_Pad_D2.0mm_ValueSilk, symbol Connector:TestPoint_Small
- removed TP16: RX, Modified:TestPoint_Pad_D2.0mm_ValueSilk, symbol Connector:TestPoint_Small
Connections:
- net GPIO0: no longer U5.12 (DIAG)
- net GPIO1: no longer R12.1, U5.10 (VL)
- net GPIO20: now also U5.12 (DIAG)
- net GPIO21: now also R12.1, U5.10 (VL); no longer U3.2 (TXD)
- net GPIO22: no longer U3.3 (RXD)
- no-connect marks 45 -> 47
Changed lines of the file:
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@@
 	)
 	(no_connect
+		(at 132.08 69.85)
+	)
+	(no_connect
 		(at 441.96 91.44)
 	)
@@
 	)
 	(no_connect
+		(at 132.08 67.31)
+	)
+	(no_connect
 		(at 143.51 27.94)
 	)
@@
 	(wire
 		(pts
-			(xy 378.46 40.64) (xy 401.32 40.64)
-		)
-		(stroke
-			(width 0)
-			(type default)
-		)
-	)
-	(wire
-		(pts
 			(xy 158.75 181.61) (xy 167.64 181.61)
 		)
@@
 	(wire
 		(pts
-			(xy 378.46 43.18) (xy 401.32 43.18)
-		)
-		(stroke
-			(width 0)
-			(type default)
-		)
-	)
-	(wire
-		(pts
 			(xy 121.92 186.69) (xy 133.35 186.69)
 		)
@@
 	(wire
 		(pts
-			(xy 132.08 67.31) (xy 148.59 67.31)
-		)
-		(stroke
-			(width 0)
-			(type default)
-		)
-	)
-	(wire
-		(pts
 			(xy 127 167.64) (xy 127 168.91)
 		)
@@
 	(wire
 		(pts
-			(xy 132.08 69.85) (xy 148.59 69.85)
-		)
-		(stroke
-			(width 0)
-			(type default)
-		)
-	)
-	(wire
-		(pts
 			(xy 129.54 175.26) (xy 132.08 175.26)
 		)
@@
 		)
 	)
-	(label "GPIO1"
+	(label "GPIO21"
 		(at 340.36 50.8 0)
 		(effects
@@
 		)
 	)
-	(label "USB_SERIAL_TXO"
-		(at 148.59 67.31 180)
-		(effects
-			(font
-				(size 1.27 1.27)
-			)
-			(justify right bottom)
-		)
-	)
 	(label "GPIO26"
 		(at 509.27 83.82 0)
@@
 		)
 	)
-	(label "USB_SERIAL_TXO"
-		(at 398.78 43.18 180)
-		(effects
-			(font
-				(size 1.27 1.27)
-			)
-			(justify right bottom)
-		)
-	)
 	(label "GPIO3"
 		(at 441.96 38.1 180)
@@
 		)
 	)
-	(label "USB_SERIAL_RXI"
-		(at 148.59 69.85 180)
-		(effects
-			(font
-				(size 1.27 1.27)
-			)
-			(justify right bottom)
-		)
-	)
 	(label "SWD"
 		(at 509.27 91.44 0)
@@
 		)
 	)
-	(label "GPIO0"
+	(label "GPIO20"
 		(at 340.36 40.64 0)
 		(effects
@@
 		)
 	)
-	(label "GPIO22"
-		(at 378.46 40.64 180)
-		(effects
-			(font
-				(size 1.27 1.27)
-			)
-			(justify right bottom)
-		)
-	)
-	(label "USB_SERIAL_RXI"
-		(at 398.78 40.64 180)
-		(effects
-			(font
-				(size 1.27 1.27)
-			)
-			(justify right bottom)
-		)
-	)
 	(label "STRAIN_E-"
 		(at 121.92 191.77 0)
@@
 		)
 	)
-	(label "GPIO21"
-		(at 378.46 43.18 180)
-		(effects
-			(font
-				(size 1.27 1.27)
-			)
-			(justify right bottom)
-		)
-	)
 	(label "MAG_CLK"
 		(at 118.11 144.78 0)
@@
 					(unit 1)
 				)
-			)
-		)
-	)
-	(symbol
-		(lib_id "Connector:TestPoint_Small")
-		(at 401.32 40.64 0)
-		(unit 1)
-		(exclude_from_sim no)
-		(in_bom yes)
-		(on_board yes)
-		(dnp no)
-		(property "Reference" "TP15"
-			(at 402.5392 39.4716 0)
-			(effects
-				(font
-					(size 1.27 1.27)
-				)
-				(justify left)
-			)
-		)
-		(property "Value" "TX"
-			(at 402.59 40.64 0)
-			(effects
-				(font
-					(size 1.27 1.27)
-				)
-				(justify left)
-			)
-		)
-		(property "Footprint" "Modified:TestPoint_Pad_D2.0mm_ValueSilk"
-			(at 406.4 40.64 0)
-			(effects
-				(font
-					(size 1.27 1.27)
-				)
-				(hide yes)
-			)
-		)
-		(property "Datasheet" "~"
-			(at 406.4 40.64 0)
-			(effects
-				(font
-					(size 1.27 1.27)
-				)
-				(hide yes)
-			)
-		)
-		(property "Description" ""
-			(at 401.32 40.64 0)
-			(effects
-				(font
-					(size 1.27 1.27)
-				)
-			)
-		)
-		(pin "1"
-		)
-		(instances
-			(project ""
-				(path "/5edcefbe-9766-42c8-9529-28d0ec865573"
-					(reference "TP15")
-					(unit 1)
-				)
-			)
-		)
-	)
-	(symbol
-		(lib_id "Connector:TestPoint_Small")
-		(at 401.32 43.18 0)
-		(unit 1)
-		(exclude_from_sim no)
-		(in_bom yes)
-		(on_board yes)
-		(dnp no)
-		(property "Reference" "TP16"
-			(at 402.5392 42.0116 0)
-			(effects
-				(font
-					(size 1.27 1.27)
-				)
-				(justify left)
-			)
-		)
-		(property "Value" "RX"
-			(at 402.59 43.18 0)
-			(effects
-				(font
-					(size 1.27 1.27)
-				)
-				(justify left)
-			)
-		)
-		(property "Footprint" "Modified:TestPoint_Pad_D2.0mm_ValueSilk"
-			(at 406.4 43.18 0)
-			(effects
-				(font
-					(size 1.27 1.27)
-				)
-				(hide yes)
-			)
-		)
-		(property "Datasheet" "~"
-			(at 406.4 43.18 0)
-			(effects
-				(font
-					(size 1.27 1.27)
-				)
-				(hide yes)
-			)
-		)
-		(property "Description" ""
-			(at 401.32 43.18 0)
-			(effects
-				(font
-					(size 1.27 1.27)
-				)
-			)
-		)
-		(pin "1"
-		)
-		(instances
-			(project ""
-				(path "/5edcefbe-9766-42c8-9529-28d0ec865573"
-					(reference "TP16")
-					(unit 1)
-				)

Commit message: more layout and simplification
Parts:
- removed C28: 1uF, Capacitor_SMD:C_0603_1608Metric, symbol Device:C_Small
- removed Q2: UMH3N, Package_TO_SOT_SMD:SOT-363_SC-70-6, symbol Transistor_BJT:UMH3N
- removed R17: 10k, Resistor_SMD:R_0603_1608Metric, symbol Device:R_Small
- removed TP13: EN, Modified:TestPoint_Pad_D2.0mm_ValueSilk, symbol Connector:TestPoint_Small
- removed TP14: BOOT, Modified:TestPoint_Pad_D2.0mm_ValueSilk, symbol Connector:TestPoint_Small
Connections:
- net DTR: no longer names the net of U3.13 (~{DTR})
- net ESP32_BOOT renamed GPIO15
- net RTS: no longer names the net of U3.14 (~{RTS})
- no-connect marks 47 -> 49
Other:
- note removed: "Recommended 1uF-10uF on EN for auto-reset circuitry, per Espressif design notes."
- note removed: "Reset/Boot via USB serial"

Commit message: more layout
Connections:
- net GPIO10: no longer U4.12 (DOUT)
- net GPIO14: no longer U4.11 (PD_SCK)
- net GPIO16: now also J3.8 (Pin_8); no longer J3.3 (Pin_3)
- net GPIO17: now also J3.7 (Pin_7); no longer J3.4 (Pin_4)
- net GPIO18: now also J3.6 (Pin_6); no longer J3.5 (Pin_5)
- net GPIO19: now also J3.5 (Pin_5); no longer J3.6 (Pin_6)
- net GPIO2: now also U3.3 (RXD); no longer R11.1, U5.7 (WL)
- net GPIO20: now also J3.4 (Pin_4); no longer J3.7 (Pin_7), U5.12 (DIAG)
- net GPIO21: now also J3.3 (Pin_3)
- net GPIO22: now also U4.12 (DOUT)
- net GPIO23: now also U4.11 (PD_SCK); no longer J3.8 (Pin_8)
- net GPIO3: now also U3.2 (TXD); no longer R10.1, U5.6 (UL)
- net GPIO4: now also U5.12 (DIAG)
- new net TMC_UL: R10.1, U5.6 (UL)
- new net TMC_WL: R11.1, U5.7 (WL)
- no-connect marks 49 -> 47
Changed lines of the file:
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@@
 	)
 	(no_connect
-		(at 132.08 69.85)
-	)
-	(no_connect
 		(at 441.96 91.44)
 	)
@@
 	)
 	(no_connect
-		(at 132.08 67.31)
-	)
-	(no_connect
 		(at 143.51 27.94)
 	)
@@
 	(wire
 		(pts
+			(xy 323.85 53.34) (xy 340.36 53.34)
+		)
+		(stroke
+			(width 0)
+			(type default)
+		)
+	)
+	(wire
+		(pts
 			(xy 81.28 198.12) (xy 78.74 198.12)
 		)
@@
 	(wire
 		(pts
-			(xy 340.36 53.34) (xy 325.12 53.34)
-		)
-		(stroke
-			(width 0)
-			(type default)
-		)
-	)
-	(wire
-		(pts
 			(xy 184.15 186.69) (xy 184.15 187.96)
 		)
@@
 	(wire
 		(pts
-			(xy 340.36 55.88) (xy 325.12 55.88)
-		)
-		(stroke
-			(width 0)
-			(type default)
-		)
-	)
-	(wire
-		(pts
 			(xy 377.19 179.07) (xy 383.54 179.07)
 		)
@@
 	(wire
 		(pts
+			(xy 323.85 55.88) (xy 340.36 55.88)
+		)
+		(stroke
+			(width 0)
+			(type default)
+		)
+	)
+	(wire
+		(pts
 			(xy 30.48 229.87) (xy 30.48 234.95)
 		)
@@
 		)
 	)
+	(label "RXD"
+		(at 323.85 55.88 0)
+		(effects
+			(font
+				(size 1.27 1.27)
+			)
+			(justify left bottom)
+		)
+	)
 	(label "GPIO47_ADC7"
 		(at 509.27 30.48 0)
@@
 		)
 	)
-	(label "GPIO2"
+	(label "GPIO3"
 		(at 340.36 53.34 0)
 		(effects
@@
 		)
 	)
-	(label "GPIO14"
+	(label "GPIO23"
 		(at 378.46 68.58 180)
 		(effects
@@
 		)
 	)
-	(label "GPIO23"
+	(label "GPIO16"
 		(at 378.46 38.1 180)
 		(effects
@@
 	)
 	(label "TMC_UL"
-		(at 325.12 55.88 0)
+		(at 311.15 41.91 0)
 		(effects
 			(font
@@
 		)
 	)
+	(label "TXD"
+		(at 323.85 53.34 0)
+		(effects
+			(font
+				(size 1.27 1.27)
+			)
+			(justify left bottom)
+		)
+	)
 	(label "USB_D+"
 		(at 99.06 74.93 0)
@@
 		)
 	)
-	(label "GPIO20"
+	(label "GPIO17"
 		(at 378.46 45.72 180)
 		(effects
@@
 		)
 	)
-	(label "GPIO3"
+	(label "GPIO2"
 		(at 340.36 55.88 0)
 		(effects
@@
 		)
 	)
-	(label "GPIO20"
+	(label "GPIO4"
 		(at 340.36 40.64 0)
 		(effects
@@
 		)
 	)
-	(label "GPIO18"
+	(label "GPIO19"
 		(at 378.46 55.88 180)
 		(effects
@@
 		)
 	)
-	(label "GPIO19"
+	(label "TXD"
+		(at 132.08 67.31 0)
+		(effects
+			(font
+				(size 1.27 1.27)
+			)
+			(justify left bottom)
+		)
+	)
+	(label "GPIO18"
 		(at 378.46 50.8 180)
 		(effects
@@
 		)
 	)
-	(label "GPIO10"
+	(label "GPIO22"
 		(at 355.6 73.66 90)
 		(effects
@@
 		)
 	)
-	(label "GPIO17"
+	(label "GPIO20"
 		(at 378.46 58.42 180)
 		(effects
@@
 	)
 	(label "TMC_WL"
-		(at 325.12 53.34 0)
+		(at 311.15 44.45 0)
+		(effects
+			(font
+				(size 1.27 1.27)
+			)
+			(justify left bottom)
+		)
+	)
+	(label "RXD"
+		(at 132.08 69.85 0)
 		(effects
 			(font
@@
 		)
 	)
-	(label "GPIO16"
+	(label "GPIO21"
 		(at 378.46 63.5 180)
 		(effects

Commit message: finished layout
Connections:
- net TMC_UL is gone; now on net GPIO7: R10.1, U5.6 (UL)
- net TMC_WL is gone; now on net GPIO6: R11.1, U5.7 (WL)
- net GPIO10: now also R9.1, U5.5 (WH)
- net GPIO12: now also TP9.1, U1.8 (Z/W/CSN); no longer R14.2, TP5.1, U8.1 (SCL)
- net GPIO13: now also R16.1, TP10.1, U1.7 (B/V/SCL/CLK); no longer R13.2, TP4.1, U8.4 (SDA)
- net GPIO14: now also R15.2, TP11.1, U1.6 (A/U/SDA/DO)
- net GPIO15: now also R14.2, TP5.1, U8.1 (SCL)
- net GPIO21: no longer R12.1, U5.10 (VL)
- net GPIO24: now also R13.2, TP4.1, U8.4 (SDA)
- net GPIO4: no longer R7.1, U5.3 (UH)
- net GPIO5: now also R12.1, U5.10 (VL); no longer R8.1, U5.4 (VH)
- net GPIO6: no longer TP9.1, U1.8 (Z/W/CSN)
- net GPIO7: no longer R9.1, U5.5 (WH)
- net GPIO8: now also R7.1, U5.3 (UH); no longer R16.1, TP10.1, U1.7 (B/V/SCL/CLK)
- net GPIO9: now also R8.1, U5.4 (VH); no longer R15.2, TP11.1, U1.6 (A/U/SDA/DO)
- no-connect marks 47 -> 46
Changed lines of the file:
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@@
 	)
 	(no_connect
-		(at 441.96 91.44)
-	)
-	(no_connect
 		(at 509.27 38.1)
 	)
@@
 	(wire
 		(pts
-			(xy 323.85 53.34) (xy 340.36 53.34)
+			(xy 325.12 38.1) (xy 341.63 38.1)
 		)
 		(stroke
@@
 	(wire
 		(pts
-			(xy 378.46 66.04) (xy 398.78 66.04)
-		)
-		(stroke
-			(width 0)
-			(type default)
-		)
-	)
-	(wire
-		(pts
 			(xy 54.61 242.57) (xy 71.12 242.57)
 		)
@@
 	(wire
 		(pts
+			(xy 347.98 73.66) (xy 347.98 90.17)
+		)
+		(stroke
+			(width 0)
+			(type default)
+		)
+	)
+	(wire
+		(pts
 			(xy 81.28 77.47) (xy 83.82 77.47)
 		)
@@
 	(wire
 		(pts
-			(xy 340.36 58.42) (xy 325.12 58.42)
+			(xy 340.36 50.8) (xy 325.12 50.8)
 		)
 		(stroke
@@
 	(wire
 		(pts
-			(xy 340.36 63.5) (xy 323.85 63.5)
-		)
-		(stroke
-			(width 0)
-			(type default)
-		)
-	)
-	(wire
-		(pts
 			(xy 379.73 173.99) (xy 377.19 173.99)
 		)
@@
 	(wire
 		(pts
-			(xy 340.36 50.8) (xy 325.12 50.8)
-		)
-		(stroke
-			(width 0)
-			(type default)
-		)
-	)
-	(wire
-		(pts
 			(xy 351.79 204.47) (xy 347.98 204.47)
 		)
@@
 	(wire
 		(pts
+			(xy 325.12 48.26) (xy 340.36 48.26)
+		)
+		(stroke
+			(width 0)
+			(type default)
+		)
+	)
+	(wire
+		(pts
 			(xy 196.85 127) (xy 181.61 127)
 		)
@@
 	(wire
 		(pts
-			(xy 203.2 193.04) (xy 203.2 196.85)
+			(xy 325.12 45.72) (xy 340.36 45.72)
 		)
 		(stroke
@@
 	(wire
 		(pts
-			(xy 246.38 78.74) (xy 229.87 78.74)
+			(xy 203.2 193.04) (xy 203.2 196.85)
 		)
 		(stroke
@@
 	(wire
 		(pts
-			(xy 196.85 134.62) (xy 181.61 134.62)
+			(xy 246.38 78.74) (xy 229.87 78.74)
 		)
 		(stroke
@@
 	(wire
 		(pts
-			(xy 129.54 175.26) (xy 132.08 175.26)
+			(xy 196.85 134.62) (xy 181.61 134.62)
 		)
 		(stroke
@@
 	(wire
 		(pts
-			(xy 30.48 234.95) (xy 43.18 234.95)
+			(xy 129.54 175.26) (xy 132.08 175.26)
 		)
 		(stroke
@@
 	(wire
 		(pts
-			(xy 340.36 60.96) (xy 325.12 60.96)
+			(xy 30.48 234.95) (xy 43.18 234.95)
 		)
 		(stroke
@@
 	(wire
 		(pts
-			(xy 340.36 66.04) (xy 325.12 66.04)
-		)
-		(stroke
-			(width 0)
-			(type default)
-		)
-	)
-	(wire
-		(pts
 			(xy 224.79 207.01) (xy 229.87 207.01)
 		)
@@
 	(wire
 		(pts
-			(xy 323.85 55.88) (xy 340.36 55.88)
+			(xy 325.12 35.56) (xy 341.63 35.56)
 		)
 		(stroke
@@
 	(wire
 		(pts
+			(xy 325.12 53.34) (xy 340.36 53.34)
+		)
+		(stroke
+			(width 0)
+			(type default)
+		)
+	)
+	(wire
+		(pts
 			(xy 201.93 137.16) (xy 207.01 137.16)
 		)
@@
 	(wire
 		(pts
+			(xy 325.12 43.18) (xy 340.36 43.18)
+		)
+		(stroke
+			(width 0)
+			(type default)
+		)
+	)
+	(wire
+		(pts
 			(xy 256.54 234.95) (xy 269.24 234.95)
 		)
@@
 		)
 	)
+	(wire
+		(pts
+			(xy 325.12 55.88) (xy 340.36 55.88)
+		)
+		(stroke
+			(width 0)
+			(type default)
+		)
+	)
 	(label "STRAIN_E+"
 		(at 121.92 198.12 0)
@@
 		)
 	)
-	(label "GPIO4"
-		(at 340.36 58.42 0)
-		(effects
-			(font
-				(size 1.27 1.27)
-			)
-			(justify left bottom)
-		)
-	)
 	(label "GPIO18"
 		(at 441.96 76.2 180)
@@
 		)
 	)
-	(label "GPIO21"
-		(at 340.36 50.8 0)
-		(effects
-			(font
-				(size 1.27 1.27)
-			)
-			(justify left bottom)
-		)
-	)
 	(label "RXD"
-		(at 323.85 55.88 0)
+		(at 325.12 35.56 0)
 		(effects
 			(font
@@
 		)
 	)
+	(label "GPIO8"
+		(at 340.36 50.8 0)
+		(effects
+			(font
+				(size 1.27 1.27)
+			)
+			(justify left bottom)
+		)
+	)
 	(label "GPIO32"
 		(at 509.27 68.58 0)
@@
 	)
 	(label "TMC_VH"
-		(at 325.12 60.96 0)
+		(at 325.12 53.34 0)
 		(effects
 			(font
@@
 	)
 	(label "GPIO3"
-		(at 340.36 53.34 0)
+		(at 341.63 38.1 0)
 		(effects
 			(font
@@
 		)
 	)
-	(label "GPIO8"
-		(at 350.52 73.66 90)
-		(effects
-			(font
-				(size 1.27 1.27)
-			)
-			(justify left bottom)
-		)
-	)
 	(label "STRAIN_DO"
 		(at 355.6 96.52 90)
@@
 	)
 	(label "MAG_CSN"
-		(at 323.85 63.5 0)
+		(at 347.98 90.17 90)
 		(effects
 			(font
@@
 	)
 	(label "TMC_WH"
-		(at 325.12 66.04 0)
+		(at 325.12 55.88 0)
 		(effects
 			(font
@@
 		)
 	)
+	(label "GPIO12"
+		(at 347.98 73.66 90)
+		(effects
+			(font
+				(size 1.27 1.27)
+			)
+			(justify left bottom)
+		)
+	)
 	(label "USB_D-"
 		(at 67.31 73.66 180)
@@
 	)
 	(label "TMC_UL"
-		(at 311.15 41.91 0)
+		(at 325.12 48.26 0)
 		(effects
 			(font
@@
 	)
 	(label "TXD"
-		(at 323.85 53.34 0)
+		(at 325.12 38.1 0)
 		(effects
 			(font
@@
 		)
 	)
+	(label "GPIO10"
+		(at 340.36 55.88 0)
+		(effects
+			(font
+				(size 1.27 1.27)
+			)
+			(justify left bottom)
+		)
+	)
 	(label "GPIO6"
-		(at 340.36 63.5 0)
+		(at 340.36 45.72 0)
 		(effects
 			(font
@@
 	)
 	(label "TMC_VL"
-		(at 325.12 50.8 0)
+		(at 325.12 43.18 0)
 		(effects
 			(font
@@
 		)
 	)
+	(label "GPIO9"
+		(at 340.36 53.34 0)
+		(effects
+			(font
+				(size 1.27 1.27)
+			)
+			(justify left bottom)
+		)
+	)
 	(label "GPIO7"
-		(at 340.36 66.04 0)
+		(at 340.36 48.26 0)
 		(effects
 			(font
@@
 		)
 	)
-	(label "GPIO13"
+	(label "GPIO24"
 		(at 368.3 73.66 90)
 		(effects
@@
 	)
 	(label "TMC_UH"
-		(at 325.12 58.42 0)
+		(at 325.12 50.8 0)
 		(effects
 			(font
@@
 	)
 	(label "GPIO2"
-		(at 340.36 55.88 0)
+		(at 341.63 35.56 0)
 		(effects
 			(font
@@
 		)
 	)
+	(label "GPIO13"
+		(at 350.52 73.66 90)
+		(effects
+			(font
+				(size 1.27 1.27)
+			)
+			(justify left bottom)
+		)
+	)
 	(label "GPIO4"
 		(at 441.96 40.64 180)
@@
 		)
 	)
+	(label "GPIO14"
+		(at 353.06 73.66 90)
+		(effects
+			(font
+				(size 1.27 1.27)
+			)
+			(justify left bottom)
+		)
+	)
 	(label "GPIO37"
 		(at 509.27 55.88 0)
@@
 	)
 	(label "GPIO5"
-		(at 340.36 60.96 0)
+		(at 340.36 43.18 0)
 		(effects
 			(font
@@
 		)
 	)
-	(label "GPIO15"
-		(at 378.46 66.04 180)
-		(effects
-			(font
-				(size 1.27 1.27)
-			)
-			(justify right bottom)
-		)
-	)
 	(label "STRAIN_DO"
 		(at 256.54 185.42 180)
@@
 	)
 	(label "TMC_WL"
-		(at 311.15 44.45 0)
+		(at 325.12 45.72 0)
 		(effects
 			(font
@@
 		)
 	)
-	(label "GPIO9"
-		(at 353.06 73.66 90)
-		(effects
-			(font
-				(size 1.27 1.27)
-			)
-			(justify left bottom)
-		)
-	)
 	(label "STRAIN_E-"
 		(at 121.92 191.77 0)
@@
 		)
 	)
-	(label "GPIO12"
+	(label "GPIO15"
 		(at 365.76 73.66 90)
 		(effects

Commit message: redid routing and schematic to match GPIO pins from excel
Parts:
- removed U9: TS1117BCW33_RPG, Modified:SOT-223-3_TabPin2_GndOutIn, symbol Regulator_Linear:TS1117BCW33_RPG
- J1: symbol Connector:Conn_01x03_Male -> Connector:Conn_01x03_Pin
Connections:
- net GPIO10: now also U4.12 (DOUT); no longer R9.1, U5.5 (WH)
- net GPIO11: now also U4.11 (PD_SCK); no longer U7.2 (A)
- net GPIO12: now also R13.2, TP4.1, U8.4 (SDA); no longer TP9.1, U1.8 (Z/W/CSN)
- net GPIO13: now also R14.2, TP5.1, U8.1 (SCL); no longer R16.1, TP10.1, U1.7 (B/V/SCL/CLK)
- net GPIO14: now also U5.12 (DIAG); no longer R15.2, TP11.1, U1.6 (A/U/SDA/DO)
- net GPIO15: now also J3.8 (Pin_8); no longer R14.2, TP5.1, U8.1 (SCL)
- net GPIO16: now also J3.6 (Pin_6); no longer J3.8 (Pin_8)
- net GPIO18: now also J3.4 (Pin_4); no longer J3.6 (Pin_6)
- net GPIO2: now also R12.1, U5.10 (VL); no longer U3.3 (RXD)
- net GPIO20: now also J3.3 (Pin_3); no longer J3.4 (Pin_4)
- net GPIO21: no longer J3.3 (Pin_3)
- net GPIO22: no longer U4.12 (DOUT)
- net GPIO23: no longer U4.11 (PD_SCK)
- net GPIO24: no longer R13.2, TP4.1, U8.4 (SDA)
- net GPIO27: now also U7.2 (A)
- net GPIO28: now also R15.2, TP11.1, U1.6 (A/U/SDA/DO)
- net GPIO29: now also TP9.1, U1.8 (Z/W/CSN)
- net GPIO3: now also R8.1, U5.4 (VH); no longer U3.2 (TXD)
- net GPIO30: now also R16.1, TP10.1, U1.7 (B/V/SCL/CLK)
- net GPIO4: now also R11.1, U5.7 (WL); no longer U5.12 (DIAG)
- net GPIO5: now also R9.1, U5.5 (WH); no longer R12.1, U5.10 (VL)
- net GPIO6: now also R10.1, U5.6 (UL); no longer R11.1, U5.7 (WL)
- net GPIO7: now also R7.1, U5.3 (UH); no longer R10.1, U5.6 (UL)
- net GPIO8: now also U3.3 (RXD); no longer R7.1, U5.3 (UH)
- net GPIO9: now also U3.2 (TXD); no longer R8.1, U5.4 (VH)
- net SWCLK: no longer J9.2 (Pin_2)
- net SWD: no longer J9.4 (Pin_4)
- no-connect marks 46 -> 50
Other:
- note added: "DEBUGGER HEADERS"
- note removed: "GPIO12=MTDI. Should be 0 on boot for 3.3v built-in flash/psram on ESP32-PICO-v3-02"
- note removed: "IO2 must be 0 to enter UART download mode"
- moved on the sheet: J8, J9
